File: Kicad/DClassAmplifier/H-Bridge.sch (KiCad schematic (older format))
At the start: 2 parts

Commit message: FET Selection
Parts:
- removed U? (x2): 2EDL8024G, SON80P400X400X100-9N-1-V:SON80P400X400X100-9N-1-V, symbol 2EDL8024G:2EDL8024G
- added C? (x3): C_Small, symbol Device:C_Small
- added D?: D_Small, symbol Device:D_Small
- added Q? (x2): PHP23NQ11T,127, Package_TO_SOT_THT:TO-220-3_Vertical, symbol Device:Q_NMOS_GDS
- added R? (x4): R_Small, symbol Device:R_Small
- added U?: IR21834, Package_DIP:DIP-14_W7.62mm_Socket, symbol Driver_FET:IR21834
Connections:
- net labels added: GND, HS_SOURCE, PWM, VCC, V_BOOTSTRAP, V_DT, V_OUT
- wire segments 8 -> 35
Other:
- note added: "Bootstrap Circuit"
- note added: "Deadtime Selection"
- note added: "Gate Driver and Gates"
- note added: "Input Filtering"

Commit message: Sizing Gate Driver Components
Parts:
- removed C?: C_Small, symbol Device:C_Small
- removed R?: R_Small, symbol Device:R_Small
- C?: value C_Small -> 100nF 100V; footprint (none) -> Capacitor_SMD:C_0805_2012Metric_Pad1.18x1.45mm_HandSolder; Notes (none) -> > 20nF; PN (none) -> C2012X7R2A104K125AA
- C?: value C_Small -> 1uF; footprint (none) -> Capacitor_SMD:C_0805_2012Metric_Pad1.18x1.45mm_HandSolder; PN (none) -> CL21B105KAFNFNE
- D?: value D_Small -> US1B-13-F; footprint (none) -> Diode_SMD:D_SMA_Handsoldering
- R? (x2): value R_Small -> 10R
- R?: value R_Small -> 10R; Notes (none) -> Optional
Connections:
- net V_DT is gone; now on net GND: U?.4 (DT)
Changed lines of the file:
@@
-$Comp
-L Device:R_Small R?
-U 1 1 60FF882E
-P 6650 2725
-F 0 "R?" V 6454 2725 50  0000 C CNN
-F 1 "R_Small" V 6545 2725 50  0000 C CNN
-F 2 "" H 6650 2725 50  0001 C CNN
-F 3 "~" H 6650 2725 50  0001 C CNN
-	1    6650 2725
-	0    1    1    0
-$EndComp
 $Comp
 L Device:R_Small R?
@@
 P 6675 2150
 F 0 "R?" V 6479 2150 50  0000 C CNN
-F 1 "R_Small" V 6570 2150 50  0000 C CNN
+F 1 "10R" V 6570 2150 50  0000 C CNN
 F 2 "" H 6675 2150 50  0001 C CNN
 F 3 "~" H 6675 2150 50  0001 C CNN
@@
 P 4375 2425
 F 0 "D?" V 4421 2495 50  0000 L CNN
-F 1 "D_Small" V 4330 2495 50  0000 L CNN
-F 2 "" V 4375 2425 50  0001 C CNN
-F 3 "~" V 4375 2425 50  0001 C CNN
+F 1 "US1B-13-F" V 4330 2495 50  0000 L CNN
+F 2 "Diode_SMD:D_SMA_Handsoldering" V 4375 2425 50  0001 C CNN
+F 3 "https://www.diodes.com/assets/Datasheets/ds16008.pdf" V 4375 2425 50  0001 C CNN
 	1    4375 2425
 	0    1    -1   0
 $EndComp
-$Comp
-L Device:R_Small R?
-U 1 1 60FFD3FE
-P 3175 2800
-F 0 "R?" H 3234 2846 50  0000 L CNN
-F 1 "R_Small" H 3234 2755 50  0000 L CNN
-F 2 "" H 3175 2800 50  0001 C CNN
-F 3 "~" H 3175 2800 50  0001 C CNN
-	1    3175 2800
-	1    0    0    -1
-$EndComp
-Wire Wire Line
-	3175 2950 3175 2900
-Wire Wire Line
-	3175 2700 3175 2600
 Wire Wire Line
 	7125 2525 7125 2400
@@
 P 4375 2700
 F 0 "C?" H 4467 2746 50  0000 L CNN
-F 1 "C_Small" H 4467 2655 50  0000 L CNN
-F 2 "" H 4375 2700 50  0001 C CNN
+F 1 "100nF 100V" H 4467 2655 50  0000 L CNN
+F 2 "Capacitor_SMD:C_0805_2012Metric_Pad1.18x1.45mm_HandSolder" H 4375 2700 50  0001 C CNN
 F 3 "~" H 4375 2700 50  0001 C CNN
+F 4 "C2012X7R2A104K125AA" H 4375 2700 50  0001 C CNN "PN"
+F 5 "> 20nF" H 4375 2700 50  0001 C CNN "Notes"
 	1    4375 2700
 	-1   0    0    1
@@
 P 2825 1875
 F 0 "C?" H 2917 1921 50  0000 L CNN
-F 1 "C_Small" H 2917 1830 50  0000 L CNN
-F 2 "" H 2825 1875 50  0001 C CNN
+F 1 "1uF" H 2917 1830 50  0000 L CNN
+F 2 "Capacitor_SMD:C_0805_2012Metric_Pad1.18x1.45mm_HandSolder" H 2825 1875 50  0001 C CNN
 F 3 "~" H 2825 1875 50  0001 C CNN
+F 4 "CL21B105KAFNFNE" H 2825 1875 50  0001 C CNN "PN"
 	1    2825 1875
 	1    0    0    -1
@@
 Wire Wire Line
 	6175 1900 6700 1900
-$Comp
-L power:VDD #PWR?
-U 1 1 61055514
-P 3325 1675
-F 0 "#PWR?" H 3325 1525 50  0001 C CNN
-F 1 "VDD" H 3340 1848 50  0000 C CNN
-F 2 "" H 3325 1675 50  0001 C CNN
-F 3 "" H 3325 1675 50  0001 C CNN
-	1    3325 1675
-	1    0    0    -1
-$EndComp
-$Comp
-L power:GNDPWR #PWR?
-U 1 1 61055B03
-P 3325 2075
-F 0 "#PWR?" H 3325 1875 50  0001 C CNN
-F 1 "GNDPWR" H 3329 1921 50  0000 C CNN
-F 2 "" H 3325 2025 50  0001 C CNN
-F 3 "" H 3325 2025 50  0001 C CNN
-	1    3325 2075
-	1    0    0    -1
-$EndComp
-$Comp
-L Device:C_Small C?
-U 1 1 61056723
-P 3325 1875
-F 0 "C?" H 3417 1921 50  0000 L CNN
-F 1 "C_Small" H 3417 1830 50  0000 L CNN
-F 2 "" H 3325 1875 50  0001 C CNN
-F 3 "~" H 3325 1875 50  0001 C CNN
-	1    3325 1875
-	1    0    0    -1
-$EndComp
-Wire Wire Line
-	3325 2075 3325 1975
-Wire Wire Line
-	3325 1675 3325 1775
 $Comp
 L power:GND #PWR?
@@
 Text Label 4375 2875 0    50   ~ 0
 HS_SOURCE
-$Comp
-L Device:R_Small R?
-U 1 1 610D593B
-P 4375 2150
-F 0 "R?" H 4434 2196 50  0000 L CNN
-F 1 "R_Small" H 4434 2105 50  0000 L CNN
-F 2 "" H 4375 2150 50  0001 C CNN
-F 3 "~" H 4375 2150 50  0001 C CNN
-	1    4375 2150
-	1    0    0    -1
-$EndComp
 Wire Wire Line
 	4375 1950 4375 2050
@@
 Text Notes 5125 1375 0    50   ~ 0
 Gate Driver and Gates
+$Comp
+L Device:R_Small R?
+U 1 1 610D593B
+P 4375 2150
+F 0 "R?" H 4434 2196 50  0000 L CNN
+F 1 "10R" H 4434 2105 50  0000 L CNN
+F 2 "" H 4375 2150 50  0001 C CNN
+F 3 "~" H 4375 2150 50  0001 C CNN
+F 4 "Optional" H 4375 2150 50  0001 C CNN "Notes"
+	1    4375 2150
+	1    0    0    -1
+$EndComp
+$Comp
+L Device:R_Small R?
+U 1 1 60FF882E
+P 6650 2725
+F 0 "R?" V 6454 2725 50  0000 C CNN
+F 1 "10R" V 6545 2725 50  0000 C CNN
+F 2 "" H 6650 2725 50  0001 C CNN
+F 3 "~" H 6650 2725 50  0001 C CNN
+	1    6650 2725
+	0    1    1    0
+$EndComp
+Wire Wire Line
+	3175 2600 3175 2950
 $EndSCHEMATC

Commit message: Hierarchical Comparator Sheet
Updated Gate Driver as well
Parts:
- removed U?: IR21834, Package_DIP:DIP-14_W7.62mm_Socket, symbol Driver_FET:IR21834
- added U?: 2ED21834S06JXUMA1, 2ED21834S:2ED21834S06JXUMA1, symbol 2ED21834S:2ED21834S06JXUMA1
Connections:
- wire segments 32 -> 37
- no-connect marks 0 -> 4
Other:
- moved on the sheet: C?, Q?, R?
