File: Kicad/DClassAmplifier/InputStage.sch (KiCad schematic (older format))
At the start: 5 parts

Commit message: updates to schematic
Parts:
- added J5, J6: Conn_01x02, symbol Connector_Generic:Conn_01x02
- C10: renamed from C?; value C_Small -> 10u; footprint (none) -> Capacitor_SMD:C_0805_2012Metric_Pad1.18x1.45mm_HandSolder
- R15: renamed from R?; value R_Small -> 16k; footprint (none) -> Resistor_SMD:R_0603_1608Metric_Pad0.98x0.95mm_HandSolder
- gave numbers to parts that had none: 3
Connections:
- net GND: now also J5.2 (Pin_2), J6.2 (Pin_2)
- net SIG_IN: now also J5.1 (Pin_1)
- net VCC: now also J6.1 (Pin_1)
Changed lines of the file:
@@
 P 4500 3750
 AR Path="/610C616D/611D4AB2" Ref="U?"  Part="1"
-AR Path="/611D4178/611D4AB2" Ref="U?"  Part="1"
-F 0 "U?" H 5700 4137 60  0000 C CNN
+AR Path="/611D4178/611D4AB2" Ref="U3"  Part="1"
+F 0 "U3" H 5700 4137 60  0000 C CNN
 F 1 "MAX4016ESA+" H 5700 4031 60  0000 C CNN
 F 2 "21-0041B_8_MXM" H 5700 3990 60  0001 C CNN
@@
 P 6950 3725
 AR Path="/610C616D/611D4AB8" Ref="#PWR?"  Part="1"
-AR Path="/611D4178/611D4AB8" Ref="#PWR?"  Part="1"
-F 0 "#PWR?" H 6950 3575 50  0001 C CNN
+AR Path="/611D4178/611D4AB8" Ref="#PWR0134"  Part="1"
+F 0 "#PWR0134" H 6950 3575 50  0001 C CNN
 F 1 "VCC" H 6965 3898 50  0000 C CNN
 F 2 "" H 6950 3725 50  0001 C CNN
@@
 P 4475 4100
 AR Path="/610C616D/611D4AC0" Ref="#PWR?"  Part="1"
-AR Path="/611D4178/611D4AC0" Ref="#PWR?"  Part="1"
-F 0 "#PWR?" H 4475 3850 50  0001 C CNN
+AR Path="/611D4178/611D4AC0" Ref="#PWR0135"  Part="1"
+F 0 "#PWR0135" H 4475 3850 50  0001 C CNN
 F 1 "GND" H 4480 3927 50  0000 C CNN
 F 2 "" H 4475 4100 50  0001 C CNN
@@
 P 4475 3425
 AR Path="/610C616D/611D4ACC" Ref="R?"  Part="1"
-AR Path="/611D4178/611D4ACC" Ref="R?"  Part="1"
-F 0 "R?" H 4534 3471 50  0000 L CNN
-F 1 "R_Small" H 4534 3380 50  0000 L CNN
-F 2 "" H 4475 3425 50  0001 C CNN
+AR Path="/611D4178/611D4ACC" Ref="R15"  Part="1"
+F 0 "R15" H 4534 3471 50  0000 L CNN
+F 1 "16k" H 4534 3380 50  0000 L CNN
+F 2 "Resistor_SMD:R_0603_1608Metric_Pad0.98x0.95mm_HandSolder" H 4475 3425 50  0001 C CNN
 F 3 "~" H 4475 3425 50  0001 C CNN
 	1    4475 3425
@@
 P 4250 3275
 AR Path="/610C616D/611D4AD4" Ref="C?"  Part="1"
-AR Path="/611D4178/611D4AD4" Ref="C?"  Part="1"
-F 0 "C?" V 4021 3275 50  0000 C CNN
-F 1 "C_Small" V 4112 3275 50  0000 C CNN
-F 2 "" H 4250 3275 50  0001 C CNN
+AR Path="/611D4178/611D4AD4" Ref="C10"  Part="1"
+F 0 "C10" V 4021 3275 50  0000 C CNN
+F 1 "10u" V 4112 3275 50  0000 C CNN
+F 2 "Capacitor_SMD:C_0805_2012Metric_Pad1.18x1.45mm_HandSolder" H 4250 3275 50  0001 C CNN
 F 3 "~" H 4250 3275 50  0001 C CNN
 	1    4250 3275
@@
 Wire Wire Line
 	4475 3275 4475 3325
-Text HLabel 4075 3275 0    50   Input ~ 0
-SIG_IN
-Wire Wire Line
-	4075 3275 4150 3275
 Wire Wire Line
 	6900 3850 6925 3850
@@
 	4475 3625 4475 3750
 $Comp
-L Device:R_Small R?
+L Device:R_Small R13
 U 1 1 611D5D52
 P 3925 3750
-F 0 "R?" H 3984 3796 50  0000 L CNN
+F 0 "R13" H 3984 3796 50  0000 L CNN
 F 1 "10k" H 3984 3705 50  0000 L CNN
 F 2 "Resistor_SMD:R_0603_1608Metric_Pad0.98x0.95mm_HandSolder" H 3925 3750 50  0001 C CNN
@@
 	3925 3950 3925 4050
 $Comp
-L power:GND #PWR?
+L power:GND #PWR0136
 U 1 1 611D72EA
 P 3925 4300
-F 0 "#PWR?" H 3925 4050 50  0001 C CNN
+F 0 "#PWR0136" H 3925 4050 50  0001 C CNN
 F 1 "GND" H 3930 4127 50  0000 C CNN
 F 2 "" H 3925 4300 50  0001 C CNN
@@
 	3925 4300 3925 4250
 $Comp
-L power:VCC #PWR?
+L power:VCC #PWR0137
 U 1 1 611D7FF1
 P 3925 3600
-F 0 "#PWR?" H 3925 3450 50  0001 C CNN
+F 0 "#PWR0137" H 3925 3450 50  0001 C CNN
 F 1 "VCC" H 3940 3773 50  0000 C CNN
 F 2 "" H 3925 3600 50  0001 C CNN
@@
 	3925 3600 3925 3650
 $Comp
-L Device:R_Small R?
+L Device:R_Small R14
 U 1 1 611DA3FE
 P 3925 4150
-F 0 "R?" H 3984 4196 50  0000 L CNN
+F 0 "R14" H 3984 4196 50  0000 L CNN
 F 1 "10k" H 3984 4105 50  0000 L CNN
 F 2 "Resistor_SMD:R_0603_1608Metric_Pad0.98x0.95mm_HandSolder" H 3925 4150 50  0001 C CNN
@@
 	1    0    0    -1
 $EndComp
+$Comp
+L Connector_Generic:Conn_01x02 J6
+U 1 1 610F66ED
+P 3200 3900
+F 0 "J6" H 3280 3892 50  0000 L CNN
+F 1 "Conn_01x02" H 3280 3801 50  0000 L CNN
+F 2 "" H 3200 3900 50  0001 C CNN
+F 3 "~" H 3200 3900 50  0001 C CNN
+	1    3200 3900
+	1    0    0    -1
+$EndComp
+$Comp
+L power:GND #PWR0138
+U 1 1 610F7442
+P 3000 4000
+F 0 "#PWR0138" H 3000 3750 50  0001 C CNN
+F 1 "GND" H 3005 3827 50  0000 C CNN
+F 2 "" H 3000 4000 50  0001 C CNN
+F 3 "" H 3000 4000 50  0001 C CNN
+	1    3000 4000
+	1    0    0    -1
+$EndComp
+$Comp
+L power:VCC #PWR0139
+U 1 1 610F9BAE
+P 3000 3900
+F 0 "#PWR0139" H 3000 3750 50  0001 C CNN
+F 1 "VCC" H 3015 4073 50  0000 C CNN
+F 2 "" H 3000 3900 50  0001 C CNN
+F 3 "" H 3000 3900 50  0001 C CNN
+	1    3000 3900
+	1    0    0    -1
+$EndComp
+$Comp
+L Connector_Generic:Conn_01x02 J5
+U 1 1 6110382F
+P 3200 3300
+F 0 "J5" H 3280 3292 50  0000 L CNN
+F 1 "Conn_01x02" H 3280 3201 50  0000 L CNN
+F 2 "" H 3200 3300 50  0001 C CNN
+F 3 "~" H 3200 3300 50  0001 C CNN
+	1    3200 3300
+	1    0    0    -1
+$EndComp
+$Comp
+L power:GND #PWR0140
+U 1 1 61103835
+P 3000 3400
+F 0 "#PWR0140" H 3000 3150 50  0001 C CNN
+F 1 "GND" H 3005 3227 50  0000 C CNN
+F 2 "" H 3000 3400 50  0001 C CNN
+F 3 "" H 3000 3400 50  0001 C CNN
+	1    3000 3400
+	1    0    0    -1
+$EndComp
+Text Label 3000 3300 2    50   ~ 0
+SIG_IN
+Text HLabel 3000 3300 0    50   Input ~ 0
+SIG_IN
+Text Label 4150 3275 2    50   ~ 0
+SIG_IN
 $EndSCHEMATC
