File: Kicad/Input/LPF.sch (KiCad schematic (older format))
At the start: 16 parts, among them J5 Conn_01x02, J6 Conn_01x02

Commit message: Input PCB added
Parts:
- added CF1: 100n, Capacitor_SMD:C_0603_1608Metric_Pad1.08x0.95mm_HandSolder, symbol Device:C_Small
- gave numbers to parts that had none: 9
Connections:
- net GND: now also CF1.2
- net VCC: now also CF1.1
Changed lines of the file:
@@
 $EndDescr
 $Comp
-L Device:R_Small R?
+L Device:R_Small R6
 U 1 1 6119FD9F
 P 9925 5025
-F 0 "R?" V 9729 5025 50  0000 C CNN
+F 0 "R6" V 9729 5025 50  0000 C CNN
 F 1 "22k" V 9820 5025 50  0000 C CNN
 F 2 "Resistor_SMD:R_0603_1608Metric_Pad0.98x0.95mm_HandSolder" H 9925 5025 50  0001 C CNN
@@
 $EndComp
 $Comp
-L Device:R_Small R?
+L Device:R_Small R7
 U 1 1 611A0CB6
 P 10300 5025
-F 0 "R?" V 10104 5025 50  0000 C CNN
+F 0 "R7" V 10104 5025 50  0000 C CNN
 F 1 "620" V 10195 5025 50  0000 C CNN
 F 2 "Resistor_SMD:R_0603_1608Metric_Pad0.98x0.95mm_HandSolder" H 10300 5025 50  0001 C CNN
@@
 $EndComp
 $Comp
-L Device:C_Small C?
+L Device:C_Small C5
 U 1 1 611A751B
 P 9800 5200
-F 0 "C?" H 9892 5246 50  0000 L CNN
+F 0 "C5" H 9892 5246 50  0000 L CNN
 F 1 "4.7n" H 9892 5155 50  0000 L CNN
 F 2 "Capacitor_SMD:C_0603_1608Metric_Pad1.08x0.95mm_HandSolder" H 9800 5200 50  0001 C CNN
@@
 	9800 5300 9800 5350
 $Comp
-L power:GND #PWR?
+L power:GND #PWR0101
 U 1 1 611AAC29
 P 9800 5350
-F 0 "#PWR?" H 9800 5100 50  0001 C CNN
+F 0 "#PWR0101" H 9800 5100 50  0001 C CNN
 F 1 "GND" H 9805 5177 50  0000 C CNN
 F 2 "" H 9800 5350 50  0001 C CNN
@@
 $EndComp
 $Comp
-L Device:C_Small C?
+L Device:C_Small C3
 U 1 1 611BBE57
 P 7725 5525
-F 0 "C?" H 7817 5571 50  0000 L CNN
+F 0 "C3" H 7817 5571 50  0000 L CNN
 F 1 "5.6n" H 7817 5480 50  0000 L CNN
 F 2 "Capacitor_SMD:C_0603_1608Metric_Pad1.08x0.95mm_HandSolder" H 7725 5525 50  0001 C CNN
@@
 $EndComp
 $Comp
-L Device:R_Small R?
+L Device:R_Small R4
 U 1 1 611BC850
 P 7900 5225
-F 0 "R?" V 7704 5225 50  0000 C CNN
+F 0 "R4" V 7704 5225 50  0000 C CNN
 F 1 "10k" V 7795 5225 50  0000 C CNN
 F 2 "Resistor_SMD:R_0603_1608Metric_Pad0.98x0.95mm_HandSolder" H 7900 5225 50  0001 C CNN
@@
 $EndComp
 $Comp
-L Device:R_Small R?
+L Device:R_Small R5
 U 1 1 611BD0E0
 P 8400 5225
-F 0 "R?" V 8204 5225 50  0000 C CNN
+F 0 "R5" V 8204 5225 50  0000 C CNN
 F 1 "750" V 8295 5225 50  0000 C CNN
 F 2 "Resistor_SMD:R_0603_1608Metric_Pad0.98x0.95mm_HandSolder" H 8400 5225 50  0001 C CNN
@@
 	8600 5225 8500 5225
 $Comp
-L Device:C_Small C?
+L Device:C_Small C2
 U 1 1 611C0153
 P 7500 5325
-F 0 "C?" H 7592 5371 50  0000 L CNN
+F 0 "C2" H 7592 5371 50  0000 L CNN
 F 1 "56n" H 7592 5280 50  0000 L CNN
 F 2 "Capacitor_SMD:C_0603_1608Metric_Pad1.08x0.95mm_HandSolder" H 7500 5325 50  0001 C CNN
@@
 $EndComp
 $Comp
-L power:GND #PWR?
+L power:GND #PWR0102
 U 1 1 611C31DE
 P 7725 5700
-F 0 "#PWR?" H 7725 5450 50  0001 C CNN
+F 0 "#PWR0102" H 7725 5450 50  0001 C CNN
 F 1 "GND" H 7730 5527 50  0000 C CNN
 F 2 "" H 7725 5700 50  0001 C CNN
@@
 SIG_OUT
 $Comp
-L AD8567ARUZ:AD8567ARUZ U?
+L AD8567ARUZ:AD8567ARUZ U1
 U 1 1 61100E74
 P 5625 4825
-F 0 "U?" H 6425 5212 60  0000 C CNN
+F 0 "U1" H 6425 5212 60  0000 C CNN
 F 1 "AD8567ARUZ" H 6425 5106 60  0000 C CNN
 F 2 "AD8567ARUZ:AD8567ARUZ" H 6425 5065 60  0001 C CNN
@@
 AR Path="/610C616D/61106B01" Ref="#PWR040"  Part="1"
 AR Path="/611D4178/61106B01" Ref="#PWR?"  Part="1"
-AR Path="/6113023B/61106B01" Ref="#PWR?"  Part="1"
-F 0 "#PWR?" H 5400 4925 50  0001 C CNN
+AR Path="/6113023B/61106B01" Ref="#PWR0103"  Part="1"
+F 0 "#PWR0103" H 5400 4925 50  0001 C CNN
 F 1 "VCC" H 5415 5248 50  0000 C CNN
 F 2 "" H 5400 5075 50  0001 C CNN
@@
 AR Path="/610C616D/61106B09" Ref="#PWR041"  Part="1"
 AR Path="/611D4178/61106B09" Ref="#PWR?"  Part="1"
-AR Path="/6113023B/61106B09" Ref="#PWR?"  Part="1"
-F 0 "#PWR?" H 7350 4875 50  0001 C CNN
+AR Path="/6113023B/61106B09" Ref="#PWR0104"  Part="1"
+F 0 "#PWR0104" H 7350 4875 50  0001 C CNN
 F 1 "GND" H 7355 4952 50  0000 C CNN
 F 2 "" H 7350 5125 50  0001 C CNN
@@
 AR Path="/610C616D/61106B14" Ref="R15"  Part="1"
 AR Path="/611D4178/61106B14" Ref="R?"  Part="1"
-AR Path="/6113023B/61106B14" Ref="R?"  Part="1"
-F 0 "R?" H 4759 5921 50  0000 L CNN
+AR Path="/6113023B/61106B14" Ref="R3"  Part="1"
+F 0 "R3" H 4759 5921 50  0000 L CNN
 F 1 "16k" H 4759 5830 50  0000 L CNN
 F 2 "Resistor_SMD:R_0603_1608Metric_Pad0.98x0.95mm_HandSolder" H 4700 5875 50  0001 C CNN
@@
 AR Path="/610C616D/61106B1C" Ref="C10"  Part="1"
 AR Path="/611D4178/61106B1C" Ref="C?"  Part="1"
-AR Path="/6113023B/61106B1C" Ref="C?"  Part="1"
-F 0 "C?" V 4246 6000 50  0000 C CNN
+AR Path="/6113023B/61106B1C" Ref="C1"  Part="1"
+F 0 "C1" V 4246 6000 50  0000 C CNN
 F 1 "10u" V 4337 6000 50  0000 C CNN
 F 2 "Capacitor_SMD:C_0805_2012Metric_Pad1.18x1.45mm_HandSolder" H 4475 6000 50  0001 C CNN
@@
 AR Path="/611D4178/61106B32" Ref="R?"  Part="1"
 AR Path="/610C616D/61106B32" Ref="R13"  Part="1"
-AR Path="/6113023B/61106B32" Ref="R?"  Part="1"
-F 0 "R?" H 4484 4871 50  0000 L CNN
+AR Path="/6113023B/61106B32" Ref="R1"  Part="1"
+F 0 "R1" H 4484 4871 50  0000 L CNN
 F 1 "10k" H 4484 4780 50  0000 L CNN
 F 2 "Resistor_SMD:R_0603_1608Metric_Pad0.98x0.95mm_HandSolder" H 4425 4825 50  0001 C CNN
@@
 AR Path="/611D4178/61106B3C" Ref="#PWR?"  Part="1"
 AR Path="/610C616D/61106B3C" Ref="#PWR039"  Part="1"
-AR Path="/6113023B/61106B3C" Ref="#PWR?"  Part="1"
-F 0 "#PWR?" H 4425 5125 50  0001 C CNN
+AR Path="/6113023B/61106B3C" Ref="#PWR0105"  Part="1"
+F 0 "#PWR0105" H 4425 5125 50  0001 C CNN
 F 1 "GND" H 4430 5202 50  0000 C CNN
 F 2 "" H 4425 5375 50  0001 C CNN
@@
 AR Path="/611D4178/61106B43" Ref="#PWR?"  Part="1"
 AR Path="/610C616D/61106B43" Ref="#PWR038"  Part="1"
-AR Path="/6113023B/61106B43" Ref="#PWR?"  Part="1"
-F 0 "#PWR?" H 4425 4525 50  0001 C CNN
+AR Path="/6113023B/61106B43" Ref="#PWR0106"  Part="1"
+F 0 "#PWR0106" H 4425 4525 50  0001 C CNN
 F 1 "VCC" H 4440 4848 50  0000 C CNN
 F 2 "" H 4425 4675 50  0001 C CNN
@@
 AR Path="/611D4178/61106B4A" Ref="R?"  Part="1"
 AR Path="/610C616D/61106B4A" Ref="R14"  Part="1"
-AR Path="/6113023B/61106B4A" Ref="R?"  Part="1"
-F 0 "R?" H 4484 5271 50  0000 L CNN
+AR Path="/6113023B/61106B4A" Ref="R2"  Part="1"
+F 0 "R2" H 4484 5271 50  0000 L CNN
 F 1 "10k" H 4484 5180 50  0000 L CNN
 F 2 "Resistor_SMD:R_0603_1608Metric_Pad0.98x0.95mm_HandSolder" H 4425 5225 50  0001 C CNN
@@
 AR Path="/611D4178/61106B50" Ref="J?"  Part="1"
 AR Path="/610C616D/61106B50" Ref="J6"  Part="1"
-AR Path="/6113023B/61106B50" Ref="J?"  Part="1"
-F 0 "J?" H 1530 3942 50  0000 L CNN
+AR Path="/6113023B/61106B50" Ref="J2"  Part="1"
+F 0 "J2" H 1530 3942 50  0000 L CNN
 F 1 "Conn_01x02" H 1530 3851 50  0000 L CNN
 F 2 "TerminalBlock:TerminalBlock_bornier-2_P5.08mm" H 1450 3950 50  0001 C CNN
@@
 AR Path="/611D4178/61106B56" Ref="#PWR?"  Part="1"
 AR Path="/610C616D/61106B56" Ref="#PWR037"  Part="1"
-AR Path="/6113023B/61106B56" Ref="#PWR?"  Part="1"
-F 0 "#PWR?" H 1250 3800 50  0001 C CNN
+AR Path="/6113023B/61106B56" Ref="#PWR0107"  Part="1"
+F 0 "#PWR0107" H 1250 3800 50  0001 C CNN
 F 1 "GND" H 1255 3877 50  0000 C CNN
 F 2 "" H 1250 4050 50  0001 C CNN
@@
 AR Path="/611D4178/61106B5C" Ref="#PWR?"  Part="1"
 AR Path="/610C616D/61106B5C" Ref="#PWR036"  Part="1"
-AR Path="/6113023B/61106B5C" Ref="#PWR?"  Part="1"
-F 0 "#PWR?" H 1250 3800 50  0001 C CNN
+AR Path="/6113023B/61106B5C" Ref="#PWR0108"  Part="1"
+F 0 "#PWR0108" H 1250 3800 50  0001 C CNN
 F 1 "VCC" H 1265 4123 50  0000 C CNN
 F 2 "" H 1250 3950 50  0001 C CNN
@@
 AR Path="/611D4178/61106B62" Ref="J?"  Part="1"
 AR Path="/610C616D/61106B62" Ref="J5"  Part="1"
-AR Path="/6113023B/61106B62" Ref="J?"  Part="1"
-F 0 "J?" H 1530 3342 50  0000 L CNN
+AR Path="/6113023B/61106B62" Ref="J1"  Part="1"
+F 0 "J1" H 1530 3342 50  0000 L CNN
 F 1 "Conn_01x02" H 1530 3251 50  0000 L CNN
 F 2 "TerminalBlock:TerminalBlock_bornier-2_P5.08mm" H 1450 3350 50  0001 C CNN
@@
 AR Path="/611D4178/61106B68" Ref="#PWR?"  Part="1"
 AR Path="/610C616D/61106B68" Ref="#PWR035"  Part="1"
-AR Path="/6113023B/61106B68" Ref="#PWR?"  Part="1"
-F 0 "#PWR?" H 1250 3200 50  0001 C CNN
+AR Path="/6113023B/61106B68" Ref="#PWR0109"  Part="1"
+F 0 "#PWR0109" H 1250 3200 50  0001 C CNN
 F 1 "GND" H 1255 3277 50  0000 C CNN
 F 2 "" H 1250 3450 50  0001 C CNN
@@
 	7250 4825 7225 4825
 $Comp
-L Device:C_Small C?
+L Device:C_Small C4
 U 1 1 611A7CBC
 P 9700 4925
-F 0 "C?" H 9792 4971 50  0000 L CNN
+F 0 "C4" H 9792 4971 50  0000 L CNN
 F 1 "47n" H 9792 4880 50  0000 L CNN
 F 2 "Capacitor_SMD:C_0603_1608Metric_Pad1.08x0.95mm_HandSolder" H 9700 4925 50  0001 C CNN
@@
 AR Path="/6110E8F0" Ref="TP?"  Part="1"
 AR Path="/610C616D/6110E8F0" Ref="TP10"  Part="1"
-AR Path="/6113023B/6110E8F0" Ref="TP?"  Part="1"
-F 0 "TP?" H 5683 5843 50  0000 L CNN
+AR Path="/6113023B/6110E8F0" Ref="TP5"  Part="1"
+F 0 "TP5" H 5683 5843 50  0000 L CNN
 F 1 "TestPoint" H 5683 5752 50  0000 L CNN
 F 2 "TestPoint:TestPoint_Pad_D2.0mm" H 5825 5725 50  0001 C CNN
@@
 	1    0    0    -1
 $EndComp
+$Comp
+L Device:C_Small C?
+U 1 1 61160214
+P 5400 5225
+AR Path="/610C616D/61160214" Ref="C?"  Part="1"
+AR Path="/611D4178/61160214" Ref="C?"  Part="1"
+AR Path="/6113023B/61160214" Ref="CF1"  Part="1"
+F 0 "CF1" V 5171 5225 50  0000 C CNN
+F 1 "100n" V 5262 5225 50  0000 C CNN
+F 2 "Capacitor_SMD:C_0603_1608Metric_Pad1.08x0.95mm_HandSolder" H 5400 5225 50  0001 C CNN
+F 3 "~" H 5400 5225 50  0001 C CNN
+	1    5400 5225
+	1    0    0    -1
+$EndComp
+Connection ~ 5400 5125
+$Comp
+L power:GND #PWR0119
+U 1 1 61165F28
+P 5400 5325
+F 0 "#PWR0119" H 5400 5075 50  0001 C CNN
+F 1 "GND" H 5405 5152 50  0000 C CNN
+F 2 "" H 5400 5325 50  0001 C CNN
+F 3 "" H 5400 5325 50  0001 C CNN
+	1    5400 5325
+	1    0    0    -1
+$EndComp
